File: Hardware/Electrical-Schematics/Vanity_Mirror_Project.kicad_sch (KiCad schematic)
At the start: 41 parts, among them IC1 SN74LV1T34QDBVRQ1, IC2 FDC1004QDGSRQ1, J1 USB_C_Receptacle_USB2.0_14P, Q1 Q_NPN_BEC, Q2 Q_NPN_BEC, SW1 RST, U1 CH340C, U2 ESP-12F, U3 USBLC6-2SC6, U4 XL1509-3.3

Commit message: 2nd version of the design
Changed multiple footprints to smd parts, Made a 2nd version for the PCB utilizing a power plane. PCB is ready to be manufactured
Parts:
- removed D1: 1N5820, Diode_THT:D_DO-201AD_P15.24mm_Horizontal, symbol Diode:1N5820
- removed J1: USB_C_Receptacle_USB2.0_14P, Connector_USB:USB_C_Receptacle_GCT_USB4085, symbol Connector:USB_C_Receptacle_USB2.0_14P
- removed R1, R4: 10k, Resistor_SMD:R_0603_1608Metric, symbol Device:R
- removed U2: ESP-12F, RF_Module:ESP-12E, symbol RF_Module:ESP-12F
- added D2: Diode, VanityMirror_FootPrints:P27_DO-214AB_SMC, symbol VanityMirror_Symbols:Diode
- added Je1: 10155435-00011LF-Custom, VanityMirror_FootPrints:2130830005_MOL, symbol Connector:USB_C_Receptacle_USB2.0_16P
- added U5: ESP32-C3-WROOM-02-N4, VanityMirror_FootPrints:MODULE_ESP32-C3-WROOM-02-H4, symbol VanityMirror_Symbols:ESP32-C3-WROOM-02-N4
- added Ur1: CPDQR5V0U, VanityMirror_FootPrints:CPDQR, symbol VanityMirror_Symbols:CPDQR5V0U
- C10: value 470uF -> 330uF
- Q1, Q2: footprint VanityMirror_FootPrints:PMEG2020EPASX -> VanityMirror_FootPrints:SOT-23-3_1P4X3P040_ONS
- R11: value 10k -> 499
- SW1: footprint Button_Switch_THT:SW_PUSH_1P1T_6x3.5mm_H4.3_APEM_MJTP1243 -> Button_Switch_SMD:SW_Push_SPST_NO_Alps_SKRK
Connections:
- net +3.3V: now also U5.1 (3V3); no longer R11.1
- net GND: now also D2.1 (A), Je1.A1 (GND), Je1.A12 (GND), Je1.A8 (SBU1), Je1.B1 (GND), Je1.B12 (GND), Je1.B8 (SBU2), Je1.SH (SHIELD), U5.19 (GND__1), U5.20 (GND__2), U5.21 (GND__3), U5.22 (GND__4), U5.23 (GND__5), U5.24 (GND__6), U5.25 (GND__7), U5.26 (GND__8), U5.27 (GND__9), U5.28 (GND__10), U5.29 (GND__11), U5.30 (GND__12), U5.31 (GND__13), U5.32 (GND__14), U5.33 (GND__15), U5.34 (GND__16), U5.35 (GND__17), U5.36 (GND__18), U5.37 (GND__19), U5.38 (GND__20), U5.39 (GND__21), U5.9 (GND), Ur1.2
- net GPIO0: now also U5.18 (IO0); no longer R11.2
- net RX: now also U5.11 (RXD)
- net SCL: now also U5.5 (IO6)
- net SDA: now also U5.6 (IO7)
- net SN74_1A: now also U5.4 (IO5)
- net TX: now also R11.2
- net at C4.1, F2.1, U3.5 (VBUS): now also Je1.A4 (VBUS), Je1.A9 (VBUS), Je1.B4 (VBUS), Je1.B9 (VBUS), Ur1.1
- net at L2.1, U4.2 (OUT): now also D2.2 (C)
- net at U3.1 (I/O1): now also Je1.A6 (D+), Je1.B6 (D+)
- net at U3.3 (I/O2): now also Je1.A7 (D-), Je1.B7 (D-)
- net at R5.2: now also Je1.A5 (CC1)
- net at R6.2: now also Je1.B5 (CC2)
- net ~{RST} renamed EN
- net EN: now also U5.2 (EN)
- new net: R11.1, U5.12 (TXD)
- no-connect marks 15 -> 14
Other:
- moved on the sheet: C1, C2, C4, F2, LED_Pins1, R5, R6, R7, R8, SW1, U3
